Commit message: Implement Unitree Go2's xacro in gazebo_ros

File: src/go2_description/xacro/leg.xacro (robot description, xacro)
@@ -1,5 +1,5 @@
 <?xml version="1.0"?>
 <robot xmlns:xacro="http://www.ros.org/wiki/xacro">
-    <xacro:include filename="$(find go2_description)/xacro/transmission.xacro"/>
+    <xacro:include filename="/home/lava-tube-mapping/src/go2_description/xacro/transmission.xacro"/>
     <xacro:macro name="leg" params="name mirror mirror_dae front_hind front_hind_dae">
         <joint name="${name}_hip_joint" type="revolute">
@@ -42,5 +42,5 @@
                 </xacro:if>
                 <geometry>
-                    <mesh filename="package://go2_description/meshes/hip.dae" scale="1 1 1"/>
+                    <mesh filename="/home/lava-tube-mapping/src/go2_description/meshes/hip.dae" scale="1 1 1"/>
                 </geometry>
                 <!-- <material name="orange"/> -->
@@ -74,8 +74,8 @@
                 <geometry>
                     <xacro:if value="${mirror_dae == True}">
-                        <mesh filename="package://go2_description/meshes/thigh.dae" scale="1 1 1"/>
+                        <mesh filename="/home/lava-tube-mapping/src/go2_description/meshes/thigh.dae" scale="1 1 1"/>
                     </xacro:if>
                     <xacro:if value="${mirror_dae == False}">
-                        <mesh filename="package://go2_description/meshes/thigh_mirror.dae" scale="1 1 1"/>
+                        <mesh filename="/home/lava-tube-mapping/src/go2_description/meshes/thigh_mirror.dae" scale="1 1 1"/>
                     </xacro:if>
                 </geometry>
@@ -109,5 +109,5 @@
                 <origin rpy="0 0 0" xyz="0 0 0"/>
                 <geometry>
-                    <mesh filename="package://go2_description/meshes/calf.dae" scale="1 1 1"/>
+                    <mesh filename="/home/lava-tube-mapping/src/go2_description/meshes/calf.dae" scale="1 1 1"/>
                 </geometry>
                 <!-- <material name="orange"/> -->

File: src/go2_description/xacro/robot.xacro (robot description, xacro)
@@ -1,10 +1,10 @@
 <?xml version="1.0"?>
-<robot name="go2" xmlns:xacro="http://www.ros.org/wiki/xacro">
+<robot xmlns:xacro="http://www.ros.org/wiki/xacro" name="go2">
     <xacro:arg name="DEBUG" default="false"/>
-    <xacro:include filename="$(find go2_description)/xacro/const.xacro"/>
-    <xacro:include filename="$(find go2_description)/xacro/materials.xacro"/>
-    <xacro:include filename="$(find go2_description)/xacro/leg.xacro"/>
-    <!-- <xacro:include filename="$(find go2_description)/xacro/stairs.xacro"/> -->
-    <xacro:include filename="$(find go2_description)/xacro/gazebo.xacro"/>
+    <xacro:include filename="/home/lava-tube-mapping/src/go2_description/xacro/const.xacro"/>
+    <xacro:include filename="/home/lava-tube-mapping/src/go2_description/xacro/materials.xacro"/>
+    <xacro:include filename="/home/lava-tube-mapping/src/go2_description/xacro/leg.xacro"/>
+    <!-- <xacro:include filename="/home/lava-tube-mapping/src/go2_description/xacro/stairs.xacro"/> -->
+    <xacro:include filename="/home/lava-tube-mapping/src/go2_description/xacro/gazebo.xacro"/>
     <!-- <xacro:include filename="$(find go2_gazebo)/launch/stairs.urdf.xacro"/> -->
     <!-- <xacro:stairs stairs="15" xpos="0" ypos="0" zpos="0" /> -->
@@ -24,5 +24,5 @@
             <origin rpy="0 0 0" xyz="0 0 0"/>
             <geometry>
-                <box size="0.001 0.001 0.001"/>
+                <mesh filename="/home/lava-tube-mapping/src/go2_description/meshes/base.dae" scale="1 1 1"/>
             </geometry>
         </visual>
@@ -37,7 +37,6 @@
             <origin rpy="0 0 0" xyz="0 0 0"/>
             <geometry>
-                <mesh filename="package://go2_description/meshes/trunk.dae" scale="1 1 1"/>
+                <mesh filename="/home/lava-tube-mapping/src/go2_description/meshes/trunk.dae" scale="1 1 1"/>
             </geometry>
-            <!-- <material name="orange"/> -->
         </visual>
         <collision>
