Commit message: Fix ros2_control and joint_state_publisher in gazebo

File: src/go2_description/xacro/gazebo.xacro (robot description, xacro)
@@ -3,7 +3,9 @@
     <!-- ros_control plugin -->
     <gazebo>
-        <plugin name="gazebo_ros_control" filename="libgazebo_ros_control.so">
-            <robotNamespace>/go2_gazebo</robotNamespace>
-            <robotSimType>gazebo_ros_control/DefaultRobotHWSim</robotSimType>
+        <plugin name="gazebo_ros2_control" filename="libgazebo_ros2_control.so">
+            <robotNamespace>go2_gazebo</robotNamespace>
+            <robotSimType>gazebo_ros2_control/DefaultRobotHWSim</robotSimType>
+            <parameters>$(find go2_description)/config/robot_control.yaml</parameters>
+            <e_stop_topic>/go2/estop</e_stop_topic>
         </plugin>
     </gazebo>
@@ -54,4 +56,21 @@
         </sensor>
     </gazebo>
+    <gazebo>
+        <plugin name="gazebo_ros_joint_state_publisher" filename="libgazebo_ros_joint_state_publisher.so">
+            <update_rate>20</update_rate>
+            <joint_name>FL_hip_joint</joint_name>
+            <joint_name>FL_thigh_joint</joint_name>
+            <joint_name>FL_calf_joint</joint_name>
+            <joint_name>FR_hip_joint</joint_name>
+            <joint_name>FR_thigh_joint</joint_name>
+            <joint_name>FR_calf_joint</joint_name>
+            <joint_name>RL_hip_joint</joint_name>
+            <joint_name>RL_thigh_joint</joint_name>
+            <joint_name>RL_calf_joint</joint_name>
+            <joint_name>RR_hip_joint</joint_name>
+            <joint_name>RR_thigh_joint</joint_name>
+            <joint_name>RR_calf_joint</joint_name>
+        </plugin>
+    </gazebo>
     <!-- Foot contacts. -->
     <gazebo reference="FR_calf">
@@ -233,3 +252,112 @@
         <kd  value="1.0"/>
     </gazebo>
+    <ros2_control name="GazeboSystem" type="system">
+        <hardware>
+            <plugin>gazebo_ros2_control/GazeboSystem</plugin>
+        </hardware>
+        <joint name="FL_hip_joint">
+            <command_interface name="position">
+                <param name="min">-1.0472</param>
+                <param name="max">30.1</param>
+            </command_interface>
+            <state_interface name="position" />
+            <state_interface name="velocity" />
+        </joint>
+        <joint name="FL_thigh_joint">
+            <command_interface name="position">
+                <param name="min">-1.0472</param>
+                <param name="max">30.1</param>
+            </command_interface>
+            <state_interface name="position" />
+            <state_interface name="velocity" />
+        </joint>
+        <joint name="FL_calf_joint">
+            <command_interface name="position">
+                <param name="min">-1.0472</param>
+                <param name="max">30.1</param>
+            </command_interface>
+            <state_interface name="position" />
+            <state_interface name="velocity" />
+        </joint>
+        <joint name="FR_hip_joint">
+            <command_interface name="position">
+                <param name="min">-1.0472</param>
+                <param name="max">30.1</param>
+            </command_interface>
+            <state_interface name="position" />
+            <state_interface name="velocity" />
+        </joint>
+        <joint name="FR_thigh_joint">
+            <command_interface name="position">
+                <param name="min">-1.0472</param>
+                <param name="max">30.1</param>
+            </command_interface>
+            <state_interface name="position" />
+            <state_interface name="velocity" />
+        </joint>
+        <joint name="FR_calf_joint">
+            <command_interface name="position">
+                <param name="min">-1.0472</param>
+                <param name="max">30.1</param>
+            </command_interface>
+            <state_interface name="position" />
+            <state_interface name="velocity" />
+        </joint>
+        <joint name="RL_hip_joint">
+            <command_interface name="position">
+                <param name="min">-1.0472</param>
+                <param name="max">30.1</param>
+            </command_interface>
+            <state_interface name="position" />
+            <state_interface name="velocity" />
+        </joint>
+        <joint name="RL_thigh_joint">
+            <command_interface name="position">
+                <param name="min">-1.0472</param>
+                <param name="max">30.1</param>
+            </command_interface>
+            <state_interface name="position" />
+            <state_interface name="velocity" />
+        </joint>
+        <joint name="RL_calf_joint">
+            <command_interface name="position">
+                <param name="min">-1.0472</param>
+                <param name="max">30.1</param>
+            </command_interface>
+            <state_interface name="position" />
+            <state_interface name="velocity" />
+        </joint>
+        <joint name="RR_hip_joint">
+            <command_interface name="position">
+                <param name="min">-1.0472</param>
+                <param name="max">30.1</param>
+            </command_interface>
+            <state_interface name="position" />
+            <state_interface name="velocity" />
+        </joint>
+        <joint name="RR_thigh_joint">
+            <command_interface name="position">
+                <param name="min">-1.0472</param>
+                <param name="max">30.1</param>
+            </command_interface>
+            <state_interface name="position" />
+            <state_interface name="velocity" />
+        </joint>
+        <joint name="RR_calf_joint">
+            <command_interface name="position">
+                <param name="min">-1.0472</param>
+                <param name="max">30.1</param>
+            </command_interface>
+            <state_interface name="position" />
+            <state_interface name="velocity" />
+        </joint>
+        <!-- <joint name="right_wheel_joint">
+            <command_interface name="velocity">
+                <param name="min">-10</param>
+                <param name="max">10</param>
+            </command_interface>
+            <state_interface name="velocity" />
+            <state_interface name="position" />
+        </joint> -->
+    </ros2_control>
 </robot>

File: src/go2_description/xacro/leg.xacro (robot description, xacro)
@@ -1,5 +1,5 @@
 <?xml version="1.0"?>
 <robot xmlns:xacro="http://www.ros.org/wiki/xacro">
-    <xacro:include filename="/home/lava-tube-mapping/src/go2_description/xacro/transmission.xacro"/>
+    <xacro:include filename="$(find go2_description)/xacro/transmission.xacro"/>
     <xacro:macro name="leg" params="name mirror mirror_dae front_hind front_hind_dae">
         <joint name="${name}_hip_joint" type="revolute">
@@ -42,5 +42,5 @@
                 </xacro:if>
                 <geometry>
-                    <mesh filename="/home/lava-tube-mapping/src/go2_description/meshes/hip.dae" scale="1 1 1"/>
+                    <mesh filename="$(find go2_description)/meshes/hip.dae" scale="1 1 1"/>
                 </geometry>
                 <!-- <material name="orange"/> -->
@@ -74,8 +74,8 @@
                 <geometry>
                     <xacro:if value="${mirror_dae == True}">
-                        <mesh filename="/home/lava-tube-mapping/src/go2_description/meshes/thigh.dae" scale="1 1 1"/>
+                        <mesh filename="$(find go2_description)/meshes/thigh.dae" scale="1 1 1"/>
                     </xacro:if>
                     <xacro:if value="${mirror_dae == False}">
-                        <mesh filename="/home/lava-tube-mapping/src/go2_description/meshes/thigh_mirror.dae" scale="1 1 1"/>
+                        <mesh filename="$(find go2_description)/meshes/thigh_mirror.dae" scale="1 1 1"/>
                     </xacro:if>
                 </geometry>
@@ -109,5 +109,5 @@
                 <origin rpy="0 0 0" xyz="0 0 0"/>
                 <geometry>
-                    <mesh filename="/home/lava-tube-mapping/src/go2_description/meshes/calf.dae" scale="1 1 1"/>
+                    <mesh filename="$(find go2_description)/meshes/calf.dae" scale="1 1 1"/>
                 </geometry>
                 <!-- <material name="orange"/> -->

File: src/go2_description/xacro/robot.xacro (robot description, xacro)
@@ -2,9 +2,9 @@
 <robot xmlns:xacro="http://www.ros.org/wiki/xacro" name="go2">
     <xacro:arg name="DEBUG" default="false"/>
-    <xacro:include filename="/home/lava-tube-mapping/src/go2_description/xacro/const.xacro"/>
-    <xacro:include filename="/home/lava-tube-mapping/src/go2_description/xacro/materials.xacro"/>
-    <xacro:include filename="/home/lava-tube-mapping/src/go2_description/xacro/leg.xacro"/>
-    <!-- <xacro:include filename="/home/lava-tube-mapping/src/go2_description/xacro/stairs.xacro"/> -->
-    <xacro:include filename="/home/lava-tube-mapping/src/go2_description/xacro/gazebo.xacro"/>
+    <xacro:include filename="$(find go2_description)/xacro/const.xacro"/>
+    <xacro:include filename="$(find go2_description)/xacro/materials.xacro"/>
+    <xacro:include filename="$(find go2_description)/xacro/leg.xacro"/>
+    <!-- <xacro:include filename="$(find go2_description)/xacro/stairs.xacro"/> -->
+    <xacro:include filename="$(find go2_description)/xacro/gazebo.xacro"/>
     <!-- <xacro:include filename="$(find go2_gazebo)/launch/stairs.urdf.xacro"/> -->
     <!-- <xacro:stairs stairs="15" xpos="0" ypos="0" zpos="0" /> -->
@@ -24,5 +24,5 @@
             <origin rpy="0 0 0" xyz="0 0 0"/>
             <geometry>
-                <mesh filename="/home/lava-tube-mapping/src/go2_description/meshes/base.dae" scale="1 1 1"/>
+                <mesh filename="$(find go2_description)/meshes/base.dae" scale="1 1 1"/>
             </geometry>
         </visual>
@@ -37,5 +37,5 @@
             <origin rpy="0 0 0" xyz="0 0 0"/>
             <geometry>
-                <mesh filename="/home/lava-tube-mapping/src/go2_description/meshes/trunk.dae" scale="1 1 1"/>
+                <mesh filename="$(find go2_description)/meshes/trunk.dae" scale="1 1 1"/>
             </geometry>
         </visual>

Commit message: Temporarily save changes

File: src/go2_description/xacro/gazebo.xacro (robot description, xacro)
@@ -56,5 +56,5 @@
         </sensor>
     </gazebo>
-    <gazebo>
+    <!-- <gazebo>
         <plugin name="gazebo_ros_joint_state_publisher" filename="libgazebo_ros_joint_state_publisher.so">
             <update_rate>20</update_rate>
@@ -72,5 +72,5 @@
             <joint_name>RR_calf_joint</joint_name>
         </plugin>
-    </gazebo>
+    </gazebo> -->
     <!-- Foot contacts. -->
     <gazebo reference="FR_calf">
@@ -263,4 +263,5 @@
             <state_interface name="position" />
             <state_interface name="velocity" />
+            <state_interface name="effort" />
         </joint>
         <joint name="FL_thigh_joint">
@@ -271,4 +272,5 @@
             <state_interface name="position" />
             <state_interface name="velocity" />
+            <state_interface name="effort" />
         </joint>
         <joint name="FL_calf_joint">
@@ -279,4 +281,5 @@
             <state_interface name="position" />
             <state_interface name="velocity" />
+            <state_interface name="effort" />
         </joint>
         <joint name="FR_hip_joint">
@@ -287,4 +290,5 @@
             <state_interface name="position" />
             <state_interface name="velocity" />
+            <state_interface name="effort" />
         </joint>
         <joint name="FR_thigh_joint">
@@ -295,4 +299,5 @@
             <state_interface name="position" />
             <state_interface name="velocity" />
+            <state_interface name="effort" />
         </joint>
         <joint name="FR_calf_joint">
@@ -303,4 +308,5 @@
             <state_interface name="position" />
             <state_interface name="velocity" />
+            <state_interface name="effort" />
         </joint>
         <joint name="RL_hip_joint">
@@ -311,4 +317,5 @@
             <state_interface name="position" />
             <state_interface name="velocity" />
+            <state_interface name="effort" />
         </joint>
         <joint name="RL_thigh_joint">
@@ -319,4 +326,5 @@
             <state_interface name="position" />
             <state_interface name="velocity" />
+            <state_interface name="effort" />
         </joint>
         <joint name="RL_calf_joint">
@@ -327,4 +335,5 @@
             <state_interface name="position" />
             <state_interface name="velocity" />
+            <state_interface name="effort" />
         </joint>
         <joint name="RR_hip_joint">
@@ -335,4 +344,5 @@
             <state_interface name="position" />
             <state_interface name="velocity" />
+            <state_interface name="effort" />
         </joint>
         <joint name="RR_thigh_joint">
@@ -343,4 +353,5 @@
             <state_interface name="position" />
             <state_interface name="velocity" />
+            <state_interface name="effort" />
         </joint>
         <joint name="RR_calf_joint">
@@ -351,13 +362,6 @@
             <state_interface name="position" />
             <state_interface name="velocity" />
-        </joint>
-        <!-- <joint name="right_wheel_joint">
-            <command_interface name="velocity">
-                <param name="min">-10</param>
-                <param name="max">10</param>
-            </command_interface>
-            <state_interface name="velocity" />
-            <state_interface name="position" />
-        </joint> -->
+            <state_interface name="effort" />
+        </joint>
     </ros2_control>
 </robot>
