Commit message: Create d435i camera link

File: ros2_ws/src/ltm_go2/ltm_go2_description/urdf/go2_description.urdf (robot description, URDF)
Before this commit: robot go2_description, 29 links, 28 joints
Links:
- added link d435_camera_link, mass 0
Joints:
- added joint d435i_camera_joint: type fixed, parent base, child d435_camera_link, origin xyz=0.308 0 0.065 rpy=0 0 0, axis 0 0 0

Commit message: Fix d435i camera position and orientation and add mesh in urdf

File: ros2_ws/src/ltm_go2/ltm_go2_description/urdf/go2_description.urdf (robot description, URDF)
Before this commit: robot go2_description, 30 links, 29 joints
Links:
- link d435_camera_link: geometry visual mesh filename=package://realsense2_description/meshes/d435.dae
Joints:
- joint d435i_camera_joint: origin xyz=0.308 0 0.065 rpy=0 0 0 -> xyz=0.325 0 0.075 rpy=-1.571 0 -1.571

Commit message: Fix d435i camera link typo

File: ros2_ws/src/ltm_go2/ltm_go2_description/urdf/go2_description.urdf (robot description, URDF)
Before this commit: robot go2_description, 30 links, 29 joints
Links:
- removed link d435_camera_link
- added link d435i_camera_link, mass 0; visual mesh filename=package://realsense2_description/meshes/d435.dae
Joints:
- joint d435i_camera_joint: child d435_camera_link -> d435i_camera_link

Commit message: Fix typos and bugs in launch realsense camera

File: ros2_ws/src/ltm_go2/ltm_go2_description/urdf/go2_description.urdf (robot description, URDF)
Before this commit: robot go2_description, 30 links, 29 joints
Joints:
- joint d435i_camera_joint: origin xyz=0.325 0 0.075 rpy=-1.571 0 -1.571 -> xyz=0.345 0 0.115 rpy=0 0 0

Commit message: Built up erroneus pointclouds in octomap in odom frame due to drift (#93)
* Create explore.launch.py

* Modify pointcloud_filter to only have crop box filter

* Add visualization to crop box filter

* Fix crop box filter dimensions

* Fix pointcloud filter

* Add ground plane segmentation

* Implement mapping using filter and fix timing issue in pointcloud_processing

* Create d435i camera link

* Fix d435i camera position and orientation and add mesh in urdf

* Create d435i_camera launch

* Edit d435i launch

* Fix d435i_camera launch file

* Add depthimage_to_pointcloud2 node

* Fix depthimage_to_pointcloud2 node in launch file

* Expand ltm_go2_driver launch file with d435i

* Fix d435i camera link typo

* Add camera pointcloud subscriber in ltm_pointcloud_filter

* Minor change in explore launch

* Fix parameter typos in ltm_pointcloud_filter

* Modify d435i_camera launch file

* Fix typos and bugs in launch realsense camera

* Create ltm_pointcloud_multiplexer

* Create launch and parameter files

* Fix failure in matching field in conversion

* Add ltm_pointcloud_mux and modify explore.launch.py

* Modify d435i_camera launch file

* Fix exploration

* Modify map reader

* Fix deadlock issue in scan procedure node

File: ros2_ws/src/ltm_go2/ltm_go2_description/urdf/go2_description.urdf (robot description, URDF)
Before this commit: robot go2_description, 29 links, 28 joints
Links:
- added link d435i_camera_link, mass 0; visual mesh filename=package://realsense2_description/meshes/d435.dae
Joints:
- added joint d435i_camera_joint: type fixed, parent base, child d435i_camera_link, origin xyz=0.345 0 0.115 rpy=0 0 0, axis 0 0 0

Commit message: Adjust urdf and rviz config

File: ros2_ws/src/ltm_go2/ltm_go2_description/urdf/go2_description.urdf (robot description, URDF)
Before this commit: robot go2_description, 30 links, 29 joints
Joints:
- joint d435i_camera_joint: origin xyz=0.345 0 0.115 rpy=0 0 0 -> xyz=0.345 0 0.110 rpy=0 0 0
